File: cpu.kicad_sch (KiCad schematic)
At the start: 46 parts, among them U1 74HC164, U10 74AHC374, U11 74LS161, U12 74AHC374, U13 74LS245, U14 74AUC2G08, U15 74AUC2G08, U16 74LS245, U17 74AHC374, U18 74AUC2G08, U19 74LS245, U2 4078, U20 74AUC2G08, U21 74AHC374, U22 74AUC2G08, U23 74AUC2G08, U24 74LS244, U25 AT28C64B-15PU, U26 74AUC2G08, U27 74AUC2G08, U28 74AUC2G08, U29 74AUC2G08, U30 74AUC2G08, U31 74AUC2G08, U32 74AUC2G08, U33 74AUC2G08, U34 74HCT238, U35 CD74HCT112E, U36 TLC555xD, U37 4555, U38 LTC-4627JD, U39 TLC555xD, U4 74LS83, U5 74LS83, U6 74AHC374, U7 AT28C64B-15PU, U8 74AUC2G08, U9 74AHC374

Commit message: Improvements
Parts:
- removed U14, U15, U18, U20, U22, U23, U26, U27, U28, U29, U30, U31, U32, U33, U8: 74AUC2G08, symbol 74xGxx:74AUC2G08
- added U14, U3, U40, U8: 74LS08, symbol 74xx:74LS08
- added U26, U27, U28: 74HC14, symbol 74xx:74HC14
Connections:
- net T4 is gone; now on net ROP: U1.6 (Q3), U2.5
- net +5V: now also U14.14 (VCC), U26.14 (VCC), U27.14 (VCC), U3.14 (VCC), U40.14 (VCC), U8.14 (VCC)
- net CLK: now also U14.10, U14.2, U14.5, U27.10, U8.10, U8.13, U8.2, U8.5; no longer U39.3 (Q)
- net GND: now also U14.7 (GND), U26.7 (GND), U27.7 (GND), U3.7 (GND), U40.7 (GND), U8.7 (GND); no longer U4.13 (C0)
- net INC: now also U1.3 (Q0), U2.2, U4.13 (C0), U14.9, U27.5, U28.1, U3.11, U40.6, U8.1
- net JUMP: now also U40.13
- net LDA: now also U3.2
- net LDB: now also U3.5
- net OA: now also U3.10
- net RA: now also U26.5, U3.8, U8.12; no longer U16.19 (CE)
- net RMDR: now also U27.3, U8.4, U8.9; no longer U25.22 (~{OE})
- net ROP: now also U14.1, U14.4, U26.1, U26.11, U26.13, U26.3, U26.9, U27.9, U3.3, U3.6, U40.11, U40.3, U40.8; no longer U24.1 (OEa), U6.1 (OE)
- net SUMA: now also U3.13, U40.2
- net SUMB: now also U40.10, U40.5
- net T5: now also U3.1, U3.12, U3.4, U3.9, U40.12, U40.4
- net T6: now also U40.1, U40.9
- net at U21.11 (Cp): now also U8.11
- net at U12.11 (Cp): now also U14.6
- net at U10.11 (Cp): now also U8.6
- net at U17.11 (Cp): now also U14.3
- net at U11.2 (CP): now also U8.8
- net at U9.11 (Cp): now also U8.3
- net at U6.11 (Cp): now also U14.8
- net RB renamed ~{RB}
- removed net RPC: U1.3 (Q0), U19.19 (CE), U2.2
- new net ~{CLK}: U27.11, U39.3 (Q)
- new net ~{RA}: U16.19 (CE), U26.6
- new net ~{RMDR}: U25.22 (~{OE}), U27.4
- new net ~{ROP}: U24.1 (OEa), U26.10, U26.12, U26.2, U26.4
- new net ~{RPC}: U19.19 (CE), U27.6, U28.2
- new net ~{RSUM}: U26.8, U27.8, U6.1 (OE)
- no-connect marks 15 -> 16
Other:
- moved on the sheet: C1, C2, C3, C4, R1, R2, R3, R4, U1, U10, U11, U12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

Commit message: Control logic changes
Parts:
- removed unit 4 of U27
- removed unit 3 of U27
- removed unit 3 of U8
- added R10, R11, R12, R5, R6, R7, R8, R9: 100K, symbol Device:R
- added U15: CD74HCT283E, N16, symbol 2024-11-21_00-35-36:CD74HCT283E
- added U18: 74HC14, symbol 74xx:74HC14
- added U20: 74LS08, symbol 74xx:74LS08
Connections:
- net RESET is gone; now on net +5V: U11.1 (~{MR})
- net +5V: now also U13.19 (CE), U18.14 (VCC)
- net B1[0]: now also U19.18 (B0)
- net B1[1]: now also U19.17 (B1)
- net B1[2]: now also U19.16 (B2)
- net B1[3]: now also U19.15 (B3)
- net B1[4]: no longer U19.18 (B0)
- net B1[5]: no longer U19.17 (B1)
- net B1[6]: no longer U19.16 (B2)
- net B1[7]: no longer U19.15 (B3)
- net B[0]: now also R12.1
- net B[1]: now also R11.1
- net B[2]: now also R10.1
- net B[3]: now also R9.1
- net B[4]: now also R8.1
- net B[5]: now also R7.1
- net B[6]: now also R6.1
- net B[7]: now also R5.1
- net CLK: no longer U25.20 (~{CE})
- net GND: now also U25.20 (~{CE}), R10.2, R11.2, R12.2, R5.2, R6.2, R7.2, R8.2, R9.2, U18.7 (GND)
- net INC: now also U11.2 (CP); no longer U1.3 (Q0), U14.9, U2.2, U28.1, U3.11, U40.6, U8.1
- net JUMP: now also U34.9 (Y6); no longer U34.10 (Y5)
- net RA: now also U18.5, U20.8
- net ROP: now also U18.3; no longer U1.6 (Q3), U11.9 (~{PE}), U2.5
- net T5: now also U20.9
- net ~{RB}: now also U18.6; no longer U13.19 (CE)
- net ~{ROP}: no longer U26.10
- net ~{RSUM}: now also U26.10
- net at U24.17 (I3b): no longer U10.19 (O7)
- net OA renamed OUTA
- new net OUTB: U20.10, U34.10 (Y5)
- new net RPC: U1.3 (Q0), U2.2, U28.1, U8.1
- new net T4: U1.6 (Q3), U2.5
- new net WSUM: U14.9, U3.11, U40.6
- new net ~{WPC}: U11.9 (~{PE}), U18.4
- no-connect marks 16 -> 17
Other:
- moved on the sheet: U10, U11, U12, U13, U14A, U14B, U14C, U16, U17, U19, U24, U25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

Commit message: Fix control logic
Parts:
- removed R10, R11, R12, R5, R6, R7, R8, R9: 100K, symbol Device:R
- removed U18, U26, U28: 74HC14, symbol 74xx:74HC14
- removed U20, U40: 74LS08, symbol 74xx:74LS08
- removed unit 2 of U27
- removed unit 7 of U27
- added unit 4 of U14
- added U18, U20: 74LS08, symbol 74xx:74LS08
- added U22, U23: 74LS14, symbol 74xx:74LS14
- added U26, U28: 74LS32, symbol 74xx:74LS32
- added unit 3 of U8
Connections:
- net +5V: now also U18.14 (VCC), U20.14 (VCC), U22.14 (VCC), U23.14 (VCC), U26.14 (VCC), U28.14 (VCC); no longer U13.19 (CE)
- net GND: now also U18.7 (GND), U20.7 (GND), U22.7 (GND), U23.7 (GND), U26.7 (GND), U28.7 (GND)
- net JUMP: now also U18.2
- net LDA: now also U3.10; no longer U3.2
- net LDB: now also U3.13; no longer U3.5
- net OUTA: now also U3.2; no longer U3.10
- net OUTB: now also U3.5
- net RA: now also U3.3, U3.6, U22.5, U22.9, U28.1, U28.2, U28.3; no longer U3.8
- net RMDR: now also U22.3
- net ROP: now also U3.11, U3.8, U14.11, U18.3, U20.3, U22.13, U26.1, U26.12, U26.13, U26.2, U26.5, U28.10, U28.4, U28.5, U28.6, U28.8, U28.9; no longer U3.3, U3.6
- net RPC: now also U22.1
- net SUMA: now also U14.13, U18.5; no longer U3.13
- net SUMB: now also U20.2, U8.10
- net T5: now also U18.1, U18.4, U8.9
- net T6: now also U14.12, U20.1
- net WSUM: now also U18.6, U26.10, U26.8, U26.9, U8.8; no longer U3.11
- net ~{RA}: now also U22.6
- net ~{RB}: now also U13.19 (CE), U22.8
- net ~{RMDR}: now also U22.4
- net ~{ROP}: now also U22.10
- net ~{RPC}: now also U22.2
- net ~{RSUM}: now also U23.6
- net ~{WPC}: now also U22.12
- new net: U23.5, U26.11
- new net: U26.3, U26.4
- new net: U22.11, U26.6
Other:
- moved on the sheet: U14E, U8E

Commit message: Use eeprom for control logic
Parts:
- removed unit 4 of U14
- removed U15: CD74HCT283E, N16, symbol 2024-11-21_00-35-36:CD74HCT283E
- removed U18, U20, U3: 74LS08, symbol 74xx:74LS08
- removed U22, U23: 74LS14, symbol 74xx:74LS14
- removed U26, U28: 74LS32, symbol 74xx:74LS32
- removed U27: 74HC14, symbol 74xx:74HC14
- removed U34: 74HCT238, symbol 74xx:74HCT238
- removed U35: CD74HCT112E, N16, symbol 2024-11-04_18-16-02:CD74HCT112E
- removed U37: 4555, symbol 4xxx_IEEE:4555
- removed U38: LTC-4627JD, Display_7Segment:LTC-4627Jx, symbol Display_Character:LTC-4627JD
- removed U4, U5: 74LS83, symbol 74xx:74LS83
- removed unit 3 of U8
- added U15, U4: CD74HCT283E, N16, symbol 2024-11-25_15-26-06:CD74HCT283E
- added U18, U3: AT28C64B-15PU, AT28C64B-15PU:DIP1555W45P254L3733H482Q28, symbol AT28C64B-15PU:AT28C64B-15PU
- added U20: 74LS139, symbol 74xx:74LS139
- added U22: HS420561K-32, symbol 2024-11-04_18-16-02:HS420561K-32
- added U5: CD74HCT112E, N16, symbol 2024-11-04_18-16-02:CD74HCT112E
Connections:
- net ~{CLK} is gone; now on net CLK: U39.3 (Q)
- net +5V: now also U15.16 (VCC), U18.27 (~{WE}), U18.28 (VCC), U20.16 (VCC), U3.27 (~{WE}), U3.28 (VCC), U4.16 (VCC), U5.10 (2~{PRE}), U5.11 (2J), U5.12 (2K), U5.14 (2~{CLR}), U5.15 (1~{CLR}), U5.16 (VCC), U5.2 (1K), U5.3 (1J), U5.4 (1~{PRE})
- net GND: now also U15.8 (GND), U18.14 (GND), U18.2 (A12), U18.20 (~{CE}), U18.22 (~{OE}), U20.1 (E), U20.8 (GND), U3.14 (GND), U3.2 (A12), U3.20 (~{CE}), U3.22 (~{OE}), U4.8 (GND), U5.8 (GND)
- net INC: now also U3.17 (I/O5), U4.7 (CIN); no longer U1.5 (Q2), U2.4
- net INST0: now also U18.25 (A8), U3.25 (A8)
- net INST1: now also U18.24 (A9), U3.24 (A9)
- net INST2: now also U18.21 (A10), U3.21 (A10)
- net ROP: now also U3.18 (I/O6); no longer U14.1, U14.4
- net T4: now also U18.7 (A3), U3.7 (A3)
- net T5: now also U18.6 (A4), U3.6 (A4)
- net T6: now also U18.5 (A5), U3.5 (A5)
- net T7: now also U18.4 (A6), U3.4 (A6)
- net T8: now also U18.3 (A7), U3.3 (A7)
- net WSUM: now also U18.16 (I/O4)
- net ~{RA}: now also U18.12 (I/O1)
- net ~{RB}: now also U18.15 (I/O3)
- net ~{RMDR}: now also U3.15 (I/O3)
- net ~{RPC}: now also U3.12 (I/O1)
- net ~{RSUM}: now also U18.17 (I/O5)
- net ~{WPC}: now also U3.11 (I/O0)
- net at U36.3 (Q): now also U5.1 (1CLK)
- net at U6.18 (D7): now also U15.10 (S3)
- net at U6.17 (D6): now also U15.13 (S2)
- net at U6.14 (D5): now also U15.1 (S1)
- net at U6.13 (D4): now also U15.4 (S0)
- net at U24.17 (I3b): now also U10.19 (O7)
- net INST3: now reaches U24.3 (O3b)
- net INST3: now also U18.23 (A11), U3.23 (A11)
- net at U7.11 (I/O0): now also U22.11 (A)
- net at U7.12 (I/O1): now also U22.7 (B)
- net at U7.13 (I/O2): now also U22.4 (C)
- net at U7.15 (I/O3): now also U22.2 (D)
- net at U7.16 (I/O4): now also U22.1 (E)
- net at U7.17 (I/O5): now also U22.10 (F)
- net at U7.18 (I/O6): now also U22.5 (G)
- net at U7.19 (I/O7): now also U22.3 (DP)
- net at U7.24 (A9): now also U20.2 (A0), U5.7 (2~{Q})
- net at U7.25 (A8): now also U20.3 (A1), U5.13 (2CLK), U5.6 (1~{Q})
- net at U6.3 (D0): now also U4.4 (S0)
- net at U6.4 (D1): now also U4.1 (S1)
- net at U6.7 (D2): now also U4.13 (S2)
- net at U6.8 (D3): now also U4.10 (S3)
- net RA renamed WO
- net WO: now also U3.19 (I/O7)
- net RMDR renamed T2
- net T2: now also U18.9 (A1), U3.9 (A1); no longer U8.4
- net RPC renamed T1
- net T1: now also U18.10 (A0), U3.10 (A0); no longer U8.1
- new net: U20.4 (O0), U22.12 (D1)
- new net: U20.7 (O3), U22.6 (D4)
- new net: U20.6 (O2), U22.8 (D3)
- new net: U20.5 (O1), U22.9 (D2)
- new net: U15.7 (CIN), U4.9 (COUT)
- new net T3: U1.5 (Q2), U18.8 (A2), U2.4, U3.8 (A2)
- new net WA: U14.1, U18.11 (I/O0)
- new net WB: U14.4, U18.13 (I/O2)
- new net WIR: U3.16 (I/O4), U8.4
- new net WMAR: U3.13 (I/O2), U8.1
- no-connect marks 17 -> 15
Other:
- moved on the sheet: C1, C2, C3, C4, R1, R2, R3, R4, U1, U14C, U14E, U2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
